Commit message: Update mybot.xacro

File: gazebo_rviz/mybot_description/xacro/mybot.xacro (robot description, xacro)
@@ -144,5 +144,5 @@
       <origin xyz="0.085 0 0.085" rpy="0 0 0"/>
       <geometry>
-        <!--<mesh filename="package://robot_sim_demo/models/meshes/xtion_pro_camera.dae" />-->
+        <!--<mesh filename="package://urdf_demo/camera.dae" />-->
 	<box size="0.05 0.05 0.05"/>
       </geometry>
